File: board/controllUnit-v2/pinballControlUnit.kicad_pcb (KiCad board)
At the start: 2 copper layers, 66 x 49.5 mm, 39 parts, among them J1 Conn_01x02_Male, J10 Screw_Terminal_01x02, J11 Conn_01x02_Male, J12 Conn_01x06, J2 Conn_01x04_Male, J3 Conn_01x08_Male, J4 Conn_01x08_Male, J5 Conn_01x08_Male, J6 AudioJack2, J7 Screw_Terminal_01x02, J8 Screw_Terminal_01x02, J9 Screw_Terminal_01x02, Q1 BUK9M85-60EX, Q2 BUK9M85-60EX, Q3 BUK9M85-60EX, Q4 BUK9M85-60EX, SW1 SW_Push, SW2 SW_Push, U1 MCP1802, U2 ATtiny48-AU

Commit message: V2 fertig
Parts:
- removed the J8 at (67.9, 66.0)
- removed the J9 at (67.9, 90.2)
- removed the R6 at (82.5, 68.6)
- removed the R7 at (82.5, 92.7)
- removed the R8 at (82.5, 104.8)
- added J11: Screw_Terminal_01x02, TerminalBlock_MetzConnect:TerminalBlock_MetzConnect_Type011_RT05502HBWC_1x02_P5.00mm_Horizontal, F.Cu at (67.3, 89.5)
- added J12: Screw_Terminal_01x02, TerminalBlock_MetzConnect:TerminalBlock_MetzConnect_Type011_RT05502HBWC_1x02_P5.00mm_Horizontal, F.Cu at (67.3, 101.0)
- added Q1: BSS138, Package_TO_SOT_SMD:SOT-23, F.Cu at (76.2, 71.8)
- added Q6: BUK9M85-60EX, Package_TO_SOT_SMD:LFPAK33, F.Cu at (76.2, 77.9)
- added Q7: BUK9M85-60EX, Package_TO_SOT_SMD:LFPAK33, F.Cu at (76.2, 89.3)
- added Q8: BUK9M85-60EX, Package_TO_SOT_SMD:LFPAK33, F.Cu at (76.2, 101.0)
- added R11: 10k, Resistor_SMD:R_0805_2012Metric, F.Cu at (82.2, 83.8)
- added R12: 10k, Resistor_SMD:R_0805_2012Metric, F.Cu at (82.2, 87.6)
- added R13: 10k, Resistor_SMD:R_0805_2012Metric, F.Cu at (82.2, 91.4)
- added R14: 10k, Resistor_SMD:R_0805_2012Metric, F.Cu at (82.2, 81.9)
- added R15: 10k, Resistor_SMD:R_0805_2012Metric, F.Cu at (82.2, 85.7)
- added R16: 10k, Resistor_SMD:R_0805_2012Metric, F.Cu at (82.2, 89.5)
- added R17: 10k, Resistor_SMD:R_0805_2012Metric, F.Cu at (82.2, 93.3)
- Q2, Q3, Q4: value BUK9M85-60EX -> BSS138; footprint Package_TO_SOT_SMD:LFPAK33 -> Package_TO_SOT_SMD:SOT-23
- moved J10 24.1 mm to (67.3, 78.1)
- moved Q2 15.6 mm to (76.2, 83.2), turned to 270 degrees
- moved Q5 13.7 mm to (76.2, 66.7)
- moved J9 11.4 mm to (67.3, 66.7)
- moved Q3 4.07 mm to (76.2, 94.6), turned to 270 degrees
- moved Q4 3.70 mm to (76.2, 106.0), turned to 270 degrees
- moved R10 0.70 mm to (82.2, 80.0), turned to 0 degrees
- renumbered C2 to C1, C3 to C2, C1 to C3, D3 to D1, D1 to D2, D2 to D3, J11 to J7, J12 to J8, J7 to J9, Q1 to Q5, R13 to R1, R5 to R10, R4 to R3, R9 to R4, R1 to R5, R10 to R6, R11 to R7, R12 to R8, R3 to R9, U2 to U1, U1 to U2
Connections:
- Q2 pad 1: GND -> FET2
- Q2 pad 3: GND -> Net-(Q2-Pad3)
- Q3 pad 1: GND -> FET3
- Q3 pad 3: GND -> Net-(Q3-Pad3)
- Q4 pad 1: GND -> FET4
- Q4 pad 3: GND -> Net-(Q4-Pad3)
- Q5 pad 4: FET1 -> Net-(Q1-Pad3)
- R10 pad 2: +5V -> +3V3
- U2 pad 4: Net-(U1-Pad4) -> (no net)
Routing:
- net +3V3: track 93.4 -> 117.5 mm
- net Net-(Q4-Pad3): track 0.00 -> 21.1 mm
- net +5V: track 58.0 -> 36.9 mm
- net Net-(Q1-Pad3): track 0.00 -> 16.2 mm
- net Net-(Q3-Pad3): track 0.00 -> 13.9 mm
- net FET2: track 35.8 -> 47.6 mm
- net Net-(Q2-Pad3): track 0.00 -> 11.0 mm
- net RESET: track 60.7 -> 51.6 mm, vias 0 -> 1
- net FET1: track 39.7 -> 48.6 mm
- net RX: track 39.9 -> 32.9 mm
- net FET3: track 25.3 -> 30.6 mm
- net FET4: track 35.0 -> 39.0 mm
- net GND: track 15.3 -> 12.7 mm, vias 10 -> 7
- net PA1: track 17.0 -> 17.6 mm
- added copper zone on F.Cu, net Net-(J11-Pad1)
- added copper zone on F.Cu, net Net-(J12-Pad1)
- removed copper zone on F.Cu, net Net-(J8-Pad1) (its old number)
- removed copper zone on F.Cu, net Net-(J9-Pad1) (its old number)
Other:
- board size 66 x 49.5 mm -> 66 x 48.3 mm
- board text added: "Coil"
- board text removed: "<-Drain"
- board text removed: "<-Source"
