File: board/controllUnit-v2/pinballControlUnit.kicad_pcb (KiCad board)
At the start: 2 copper layers, 111.8 x 48.9 mm, 80 parts, among them J1 Conn_01x02_Male, J10 Screw_Terminal_01x02, J11 Screw_Terminal_01x02, J12 Screw_Terminal_01x02, J2 Conn_01x04_Male, J3 Conn_01x08_Male, J4 Conn_01x08_Male, J5 Conn_01x08_Male, J6 AudioJack2, J7 Conn_01x02_Male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

Commit message: Update pinballControlUnit.kicad_pcb
Änderungen Simon Burkhardt
Routing:
- net GND: vias 20 -> 45
Changed lines of the file:
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@@
     (thickness 1.6)
     (drawings 17)
-    (tracks 519)
+    (tracks 544)
     (zones 0)
     (modules 80)
@@
   (via (at 119.38 67.31) (size 1.6) (drill 0.8) (layers F.Cu B.Cu) (net 1))
   (via (at 110.49 104.14) (size 1.6) (drill 0.8) (layers F.Cu B.Cu) (net 1))
+  (via (at 64.135 83.185) (size 1.6) (drill 0.8) (layers F.Cu B.Cu) (net 1))
+  (via (at 77.47 83.185) (size 1.6) (drill 0.8) (layers F.Cu B.Cu) (net 1))
+  (via (at 50.8 83.185) (size 1.6) (drill 0.8) (layers F.Cu B.Cu) (net 1))
+  (via (at 37.465 83.185) (size 1.6) (drill 0.8) (layers F.Cu B.Cu) (net 1))
+  (via (at 74.93 80.01) (size 1.6) (drill 0.8) (layers F.Cu B.Cu) (net 1))
+  (via (at 74.93 81.915) (size 1.6) (drill 0.8) (layers F.Cu B.Cu) (net 1))
+  (via (at 74.93 83.82) (size 1.6) (drill 0.8) (layers F.Cu B.Cu) (net 1))
+  (via (at 61.595 80.01) (size 1.6) (drill 0.8) (layers F.Cu B.Cu) (net 1))
+  (via (at 61.595 81.915) (size 1.6) (drill 0.8) (layers F.Cu B.Cu) (net 1))
+  (via (at 61.595 83.82) (size 1.6) (drill 0.8) (layers F.Cu B.Cu) (net 1))
+  (via (at 48.26 80.01) (size 1.6) (drill 0.8) (layers F.Cu B.Cu) (net 1))
+  (via (at 48.26 81.915) (size 1.6) (drill 0.8) (layers F.Cu B.Cu) (net 1))
+  (via (at 48.26 83.82) (size 1.6) (drill 0.8) (layers F.Cu B.Cu) (net 1))
+  (via (at 39.37 80.01) (size 1.6) (drill 0.8) (layers F.Cu B.Cu) (net 1))
+  (via (at 39.37 81.915) (size 1.6) (drill 0.8) (layers F.Cu B.Cu) (net 1))
+  (via (at 39.37 83.82) (size 1.6) (drill 0.8) (layers F.Cu B.Cu) (net 1))
+  (via (at 79.375 80.01) (size 1.6) (drill 0.8) (layers F.Cu B.Cu) (net 1))
+  (via (at 79.375 81.915) (size 1.6) (drill 0.8) (layers F.Cu B.Cu) (net 1))
+  (via (at 79.375 83.82) (size 1.6) (drill 0.8) (layers F.Cu B.Cu) (net 1))
+  (via (at 66.04 80.01) (size 1.6) (drill 0.8) (layers F.Cu B.Cu) (net 1))
+  (via (at 66.04 81.915) (size 1.6) (drill 0.8) (layers F.Cu B.Cu) (net 1))
+  (via (at 66.04 83.82) (size 1.6) (drill 0.8) (layers F.Cu B.Cu) (net 1))
+  (via (at 52.705 81.915) (size 1.6) (drill 0.8) (layers F.Cu B.Cu) (net 1))
+  (via (at 52.705 83.82) (size 1.6) (drill 0.8) (layers F.Cu B.Cu) (net 1))
+  (via (at 52.705 80.01) (size 1.6) (drill 0.8) (layers F.Cu B.Cu) (net 1))
   (segment (start 103.665001 84.185001) (end 103.74 84.26) (width 0.5) (layer F.Cu) (net 2) (status 30))
   (segment (start 125.73 74.295) (end 122.2225 74.295) (width 0.5) (layer F.Cu) (net 2) (status 30))
