File: board/controllUnit-v2/pinballControlUnit.sch (KiCad schematic (older format))
At the start: 39 parts, among them J1 Conn_01x02_Male, J10 Screw_Terminal_01x02, J11 Conn_01x02_Male, J12 Conn_01x06, J2 Conn_01x04_Male, J3 Conn_01x08_Male, J4 Conn_01x08_Male, J5 Conn_01x08_Male, J6 AudioJack2, J7 Screw_Terminal_01x02, J8 Screw_Terminal_01x02, J9 Screw_Terminal_01x02, Q1 BUK9M85-60EX, Q2 BUK9M85-60EX, Q3 BUK9M85-60EX, Q4 BUK9M85-60EX, SW1 SW_Push, SW2 SW_Push, U1 MCP1802, U2 ATtiny48-AU

Commit message: V2 fertig
Parts:
- removed J8, J9: Screw_Terminal_01x02, TerminalBlock_MetzConnect:TerminalBlock_MetzConnect_Type011_RT05502HBWC_1x02_P5.00mm_Horizontal, symbol Connector:Screw_Terminal_01x02
- removed Q2, Q3, Q4: BUK9M85-60EX, Package_TO_SOT_SMD:LFPAK33, symbol Transistor_FET:BUK9M85-60EX
- removed R6, R7, R8: 10k, Resistor_SMD:R_0805_2012Metric, symbol Device:R
- added J11, J12: Screw_Terminal_01x02, TerminalBlock_MetzConnect:TerminalBlock_MetzConnect_Type011_RT05502HBWC_1x02_P5.00mm_Horizontal, symbol Connector:Screw_Terminal_01x02
- added Q1, Q2, Q3, Q4: BSS138, Package_TO_SOT_SMD:SOT-23, symbol Transistor_FET:BSS138
- added Q6, Q7, Q8: BUK9M85-60EX, Package_TO_SOT_SMD:LFPAK33, symbol Transistor_FET:BUK9M85-60EX
- added R11, R12, R13, R14, R15, R16, R17: 10k, Resistor_SMD:R_0805_2012Metric, symbol Device:R
- U2: renamed from U1; symbol pinballControlUnit-rescue:MCP1804x-3302xOT-mylib -> mylib:MCP1804x-3302xOT
- renumbered C2 to C1, C3 to C2, C1 to C3, D3 to D1, D1 to D2, D2 to D3, J11 to J7, J12 to J8, J7 to J9, Q1 to Q5, R13 to R1, R5 to R10, R4 to R3, R9 to R4, R1 to R5, R10 to R6, R11 to R7, R12 to R8, R3 to R9, U2 to U1
Connections:
- wire segments 114 -> 118
Other:
- note removed: "FET's for Coils"
- moved on the sheet: C2, C3, D1, D2, D3, J1, J8, J9, R1, R10, R2, R3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

Commit message: Spannungsversorgung und FETS komplett geändert
Parts:
- removed C3: 1u, Capacitor_SMD:C_0805_2012Metric, symbol Device:C
- removed D1: LED, LED_SMD:LED_0805_2012Metric, symbol Device:LED
- removed J10, J11, J12: Screw_Terminal_01x02, TerminalBlock_MetzConnect:TerminalBlock_MetzConnect_Type011_RT05502HBWC_1x02_P5.00mm_Horizontal, symbol Connector:Screw_Terminal_01x02
- removed Q1, Q2, Q3, Q4: BSS138, Package_TO_SOT_SMD:SOT-23, symbol Transistor_FET:BSS138
- removed Q5, Q6, Q7, Q8: BUK9M85-60EX, Package_TO_SOT_SMD:LFPAK33, symbol Transistor_FET:BUK9M85-60EX
- removed R1: 100, Resistor_SMD:R_0805_2012Metric, symbol Device:R
- removed R10, R11, R12, R13, R14, R15, R16, R17: 10k, Resistor_SMD:R_0805_2012Metric, symbol Device:R
- removed U2: MCP1802, Package_TO_SOT_SMD:SOT-23-5, symbol mylib:MCP1804x-3302xOT
- added C?: 2.2n, Capacitor_SMD:C_0805_2012Metric, symbol Device:C
- added C?: 47u, symbol Device:CP1
- added C?: 2.2u, Capacitor_SMD:C_0805_2012Metric, symbol Device:C
- added C?: 22u, Capacitor_SMD:C_0805_2012Metric, symbol Device:C
- added C?: 0.1u, Capacitor_SMD:C_0805_2012Metric, symbol Device:C
- added J? (x3): Screw_Terminal_01x02, TerminalBlock_MetzConnect:TerminalBlock_MetzConnect_Type011_RT05502HBWC_1x02_P5.00mm_Horizontal, symbol Connector:Screw_Terminal_01x02
- added L?: 68u, symbol Device:L
- added L?: 12u, symbol Device:L
- added R? (x8): R, Resistor_SMD:R_0805_2012Metric, symbol Device:R
- added R?: 100k, Resistor_SMD:R_0805_2012Metric, symbol Device:R
- added R?: 448k, Resistor_SMD:R_0805_2012Metric, symbol Device:R
- added R?: 49.9k, Resistor_SMD:R_0805_2012Metric, symbol Device:R
- added R?: 51k, Resistor_SMD:R_0805_2012Metric, symbol Device:R
- added R?: 22.1k, Resistor_SMD:R_0805_2012Metric, symbol Device:R
- added U?: LM5164, Package_SO:TI_SO-PowerPAD-8, symbol mylib:LM5164
- added U? (x4): STB16NF06L, symbol mylib:STB16NF06L
- added U? (x4): PM8841, symbol mylib:PM8841
- added U?: TPS560430, Package_TO_SOT_SMD:SOT-23-6_Handsoldering, symbol mylib:TPS560430
- C2: value 1u -> 2.2u
Connections:
- net labels added: +12V, +24V
- net labels removed: +5V
- wire segments 118 -> 150
Other:
- note added: "Gate Driver"
- moved on the sheet: C2, D2, D3, J1, J6, J7, J9, R2, R3, R5, R9, SW1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

Commit message: Schema aktualisiert
Parts:
- removed U?: PM8841, symbol mylib:PM8841
- added U5: PM8841, symbol pinballControlUnit-rescue:PM8841-mylib
- U10, U11, U8, U9: renamed from U?; symbol mylib:STB16NF06L -> pinballControlUnit-rescue:STB16NF06L-mylib
- U2: renamed from U?; symbol mylib:LM5164 -> pinballControlUnit-rescue:LM5164-mylib
- U3: renamed from U?; symbol mylib:TPS560430 -> pinballControlUnit-rescue:TPS560430-mylib
- U4, U6, U7: renamed from U?; symbol mylib:PM8841 -> pinballControlUnit-rescue:PM8841-mylib
- gave numbers to parts that had none: 23
Connections:
- wire segments 150 -> 149
Other:
- note removed: "Gate Driver"
- moved on the sheet: D2, D3, J10, J11, J12, J6, J7, J8, J9, R14, R15, R16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

Commit message: Schema fertig und David geschickt
Parts:
- removed R14, R16, R18, R20: R, Resistor_SMD:R_0805_2012Metric, symbol Device:R
- removed U10, U11, U8, U9: STB16NF06L, symbol pinballControlUnit-rescue:STB16NF06L-mylib
- removed U4, U5, U6, U7: PM8841, symbol pinballControlUnit-rescue:PM8841-mylib
- added U10, U11, U8, U9: STB16NF06L, Package_TO_SOT_SMD:TO-263-2, symbol mylib:STB16NF06L
- added U4, U5, U6, U7: PM8841, symbol mylib:PM8841
- R15, R17, R19, R21: value R -> 100
- U2: symbol pinballControlUnit-rescue:LM5164-mylib -> pinballControlUnit-rescue:LM5164-mylib-pinballControlUnit-rescue
- U3: symbol pinballControlUnit-rescue:TPS560430-mylib -> pinballControlUnit-rescue:TPS560430-mylib-pinballControlUnit-rescue
- renumbered D2 to D1, D3 to D2, R7 to R10, R8 to R11, R5 to R12, R9 to R13, R10 to R2, R11 to R3, R2 to R4, R4 to R5, R3 to R6, R12 to R7, R13 to R8, R6 to R9
Connections:
- wire segments 149 -> 124
- no-connect marks 0 -> 1
Other:
- moved on the sheet: R15, R17, R19, R21

Commit message: Leiterplatte gelayoutet
Parts:
- C4: footprint (none) -> Capacitor_SMD:CP_Elec_6.3x3.9
- L1, L2: footprint (none) -> Inductor_SMD:L_0805_2012Metric_Pad1.15x1.40mm_HandSolder
- U4, U5, U6, U7: footprint (none) -> Package_TO_SOT_SMD:SOT-23-5_HandSoldering
Changed lines of the file:
@@
 F 0 "L1" V 2719 6350 50  0000 C CNN
 F 1 "68u" V 2810 6350 50  0000 C CNN
-F 2 "" H 2900 6350 50  0001 C CNN
+F 2 "Inductor_SMD:L_0805_2012Metric_Pad1.15x1.40mm_HandSolder" H 2900 6350 50  0001 C CNN
 F 3 "~" H 2900 6350 50  0001 C CNN
 	1    2900 6350
@@
 F 0 "C4" H 3565 6896 50  0000 L CNN
 F 1 "47u" H 3565 6805 50  0000 L CNN
-F 2 "" H 3450 6850 50  0001 C CNN
+F 2 "Capacitor_SMD:CP_Elec_6.3x3.9" H 3450 6850 50  0001 C CNN
 F 3 "~" H 3450 6850 50  0001 C CNN
 	1    3450 6850
@@
 F 0 "L2" V 5619 6350 50  0000 C CNN
 F 1 "12u" V 5710 6350 50  0000 C CNN
-F 2 "" H 5800 6350 50  0001 C CNN
+F 2 "Inductor_SMD:L_0805_2012Metric_Pad1.15x1.40mm_HandSolder" H 5800 6350 50  0001 C CNN
 F 3 "~" H 5800 6350 50  0001 C CNN
 	1    5800 6350
@@
 F 0 "U4" H 8150 1950 50  0000 L CNN
 F 1 "PM8841" H 8550 1950 50  0000 L CNN
-F 2 "" H 8350 2050 50  0001 C CNN
+F 2 "Package_TO_SOT_SMD:SOT-23-5_HandSoldering" H 8350 2050 50  0001 C CNN
 F 3 "" H 8350 2050 50  0001 C CNN
 	1    8500 1700
@@
 F 0 "U5" H 8150 3050 50  0000 L CNN
 F 1 "PM8841" H 8550 3050 50  0000 L CNN
-F 2 "" H 8350 3150 50  0001 C CNN
+F 2 "Package_TO_SOT_SMD:SOT-23-5_HandSoldering" H 8350 3150 50  0001 C CNN
 F 3 "" H 8350 3150 50  0001 C CNN
 	1    8500 2800
@@
 F 0 "U6" H 8150 4150 50  0000 L CNN
 F 1 "PM8841" H 8550 4150 50  0000 L CNN
-F 2 "" H 8350 4250 50  0001 C CNN
+F 2 "Package_TO_SOT_SMD:SOT-23-5_HandSoldering" H 8350 4250 50  0001 C CNN
 F 3 "" H 8350 4250 50  0001 C CNN
 	1    8500 3900
@@
 F 0 "U7" H 8150 5250 50  0000 L CNN
 F 1 "PM8841" H 8550 5250 50  0000 L CNN
-F 2 "" H 8350 5350 50  0001 C CNN
+F 2 "Package_TO_SOT_SMD:SOT-23-5_HandSoldering" H 8350 5350 50  0001 C CNN
 F 3 "" H 8350 5350 50  0001 C CNN
 	1    8500 5000

Commit message: Schaltregler Layout gemäss Datenblatt angepasst
TPS560430
LM5164
Parts:
- U2: symbol pinballControlUnit-rescue:LM5164-mylib-pinballControlUnit-rescue -> mylib:LM5164
Connections:
- net GND: now also U2.9 (GND_PAD)
Changed lines of the file:
@@
 $EndComp
 $Comp
-L pinballControlUnit-rescue:LM5164-mylib-pinballControlUnit-rescue U2
+L mylib:LM5164 U2
 U 1 1 5D8778A7
 P 2050 6600
@@
 Wire Wire Line
 	8950 5000 9250 5000
+Wire Wire Line
+	1950 7200 2050 7200
+Connection ~ 2050 7200
 $EndSCHEMATC

Commit message: Schema+Layout fertig
Stückliste erstellt
Parts:
- added C10, C11, C8, C9: C, Capacitor_SMD:C_0805_2012Metric, symbol Device:C
- added D3, D4, D5, D6: D, LED_SMD:LED_0805_2012Metric, symbol Device:D
- added R14, R16, R18, R20: R, Resistor_SMD:R_0805_2012Metric, symbol Device:R
- C4: footprint Capacitor_SMD:CP_Elec_6.3x3.9 -> Capacitor_SMD:C_0805_2012Metric; symbol Device:CP1 -> Device:C
- L1: footprint Inductor_SMD:L_0805_2012Metric_Pad1.15x1.40mm_HandSolder -> myFootPrints:L_MSS1246-683MLB
- L2: footprint Inductor_SMD:L_0805_2012Metric_Pad1.15x1.40mm_HandSolder -> myFootPrints:L_SDR0403-120ML
Connections:
- net FET1: now also C8.2, D3.1 (K); no longer U4.3 (IN)
- net FET2: now also C9.2, D4.1 (K); no longer U5.3 (IN)
- net FET3: now also C10.2, D5.1 (K); no longer U6.3 (IN)
- net FET4: now also C11.2, D6.1 (K); no longer U7.3 (IN)
- net GND: now also R14.2, R16.2, R18.2, R20.2
- new net: C8.1, D3.2 (A), R14.1, U4.3 (IN)
- new net: C9.1, D4.2 (A), R16.1, U5.3 (IN)
- new net: C10.1, D5.2 (A), R18.1, U6.3 (IN)
- new net: C11.1, D6.2 (A), R20.1, U7.3 (IN)
Other:
- note added: "Coil switching"
- moved on the sheet: R15, R17, R19, R21, U10, U11, U4, U5, U6, U7, U8, U9

Commit message: Leiterplatte soweit fertig
Parts:
- removed C4: 47u, Capacitor_SMD:C_0805_2012Metric, symbol Device:C
- added C12: 100n, Capacitor_SMD:C_0805_2012Metric, symbol Device:C
- added C13, C14, C15, C16: 470n, Capacitor_SMD:C_0805_2012Metric, symbol Device:C
- added C4: 47u, Capacitor_SMD:C_Elec_6.3x5.8, symbol Device:CP1_Small
- added D10, D7, D8, D9: D, LED_SMD:LED_0805_2012Metric, symbol Device:D
- added R22: R, Resistor_SMD:R_0805_2012Metric, symbol Device:R
- added R23, R24, R25: 10, Resistor_SMD:R_0805_2012Metric, symbol Device:R
- added R26: 100, Resistor_SMD:R_0805_2012Metric, symbol Device:R
- added U12: LM4040DBZ-2.5, Package_TO_SOT_SMD:SOT-23, symbol Reference_Voltage:LM4040DBZ-2.5
- C2: footprint Capacitor_SMD:C_0805_2012Metric -> Capacitor_SMD:C_1206_3216Metric
- R15, R17, R19: value 100 -> 50
Connections:
- net +12V: now also C13.1, C14.1, C15.1, C16.1, C4.1
- net +3V3: now also R22.2; no longer U4.4 (IN_TH), U5.4 (IN_TH), U6.4 (IN_TH), U7.4 (IN_TH)
- net GND: now also C12.2, C13.2, C14.2, C15.2, C16.2, C4.2, U12.2 (A)
- net at R15.1, U8.1 (G): now also R23.1
- net at R15.2, U4.5 (OUT): now also D7.1 (K)
- net at R17.1, U9.1 (G): now also R24.1
- net at R17.2, U5.5 (OUT): now also D8.1 (K)
- net at R19.1, U10.1 (G): now also R25.1
- net at R19.2, U6.5 (OUT): now also D9.1 (K)
- net at R21.1, U11.1 (G): now also R26.1
- net at R21.2, U7.5 (OUT): now also D10.1 (K)
- new net: D7.2 (A), R23.2
- new net: D10.2 (A), R26.2
- new net: D9.2 (A), R25.2
- new net: D8.2 (A), R24.2
- new net +2V5: C12.1, R22.1, U12.1 (K), U4.4 (IN_TH), U5.4 (IN_TH), U6.4 (IN_TH), U7.4 (IN_TH)
Other:
- moved on the sheet: J10, J11, J12, J9, R15, R17, R19, R21, U10, U11, U8, U9
